File: street-sweep.kicad_pcb (KiCad board)
At the start: 2 copper layers, 110.6 x 95.2 mm, 56 parts, among them J1 PJ-320A, P1 GT-USB-7010ASV, SW10 SW_Push, SW10_r1 SW_Push, SW11 SW_Push, SW11_r1 SW_Push, SW12 SW_Push, SW12_r1 SW_Push, SW13_r1 SW_Push, SW14 SW_Push, SW14_r1 SW_Push, SW15 SW_Push, SW15_r1 SW_Push, SW16 SW_Push, SW16_r1 SW_Push, SW17 SW_Push, SW17_r1 SW_Push, SW18 SW_Push, SW18_r1 SW_Push, SW2 SW_Push, SW20 SW_Push, SW21 SW_Push, SW2_r1 SW_Push, SW3 SW_Push, SW3_r1 SW_Push, SW4 SW_Push, SW4_r1 SW_Push, SW5 SW_Push, SW5_r1 SW_Push, SW6 SW_Push, SW6_r1 SW_Push, SW7_r1 SW_Push, SW8 SW_Push, SW8_r1 SW_Push, SW9 SW_Push, SW9_r1 SW_Push, U1 CH552G

Commit message: Latest changes on STM32
Parts:
- removed D1, D10, D11, D12, D13, D14, D15, D16, D17, D2, D3, D4, D5, D6, D7, D8, D9: 1N4148, Diode_SMD:D_SOD-123
- removed J1: PJ-320A, Connector_Audio:Jack_3.5mm_PJ320D_Horizontal
- added C2: 4.7uF, Capacitor_SMD:C_0805_2012Metric, F.Cu at (85.1, 125.7)
- added C3: 1uF, Capacitor_SMD:C_0805_2012Metric, F.Cu at (73.5, 119.4)
- added C4: 4.7uF, Capacitor_SMD:C_0805_2012Metric, F.Cu at (92.8, 120.7)
- added C5: 1uF, Capacitor_SMD:C_0805_2012Metric, F.Cu at (89.1, 123.8)
- added P2: GT-USB-7010ASV, Connector_USB:USB_C_Receptacle_G-Switch_GT-USB-7010ASV, F.Cu at (139.7, 124.5)
- added R1: 5.1k, Resistor_SMD:R_0805_2012Metric, F.Cu at (135.0, 91.4)
- added R2: 5.1k, Resistor_SMD:R_0805_2012Metric, F.Cu at (140.2, 91.4)
- added SW1: RotaryEncoder_Switch, Rotary_Encoder:RotaryEncoder_Alps_EC11E-Switch_Vertical_H20mm, F.Cu at (136.3, 113.7)
- added U2: XC6206P332MR, Package_TO_SOT_SMD:SOT-23-3, F.Cu at (92.8, 123.8)
- C1: value 0.1uF -> 4.7uF; footprint Capacitor_SMD:C_0805_2012Metric_Pad1.18x1.45mm_HandSolder -> Capacitor_SMD:C_0805_2012Metric
- RSW1: footprint Button_Switch_SMD:SW_SPST_SKQG_WithoutStem -> Connector_PinHeader_2.54mm:PinHeader_1x02_P2.54mm_Vertical
- U1: value CH552G -> STM32F072C8T6; footprint CH552G:CH552G -> Package_QFP:LQFP-48_7x7mm_P0.5mm
- moved RSW1 68.6 mm to (68.6, 120.7), turned to 180 degrees
- moved U1 60.5 mm to (81.3, 118.7)
- moved C1 48.1 mm to (88.3, 114.6), turned to -90 degrees
- moved SW20 2.30 mm to (132.7, 134.0)
- moved SW17_r1 2.27 mm to (128.3, 131.4)
Connections:
- C1 pad 1: vcc -> +3.3V
- P1 pad A4: vcc -> +5V
- P1 pad A5: unconnected-(P1-PadA5) -> Net-(P1-PadA5)
- P1 pad A9: vcc -> +5V
- P1 pad B4: vcc -> +5V
- P1 pad B5: unconnected-(P1-PadB5) -> Net-(P1-PadB5)
- P1 pad B9: vcc -> +5V
- RSW1 pad 2: reset -> NRST
- SW10 pad 2: Row1 -> gnd
- SW10_r1 pad 2: Row1 -> gnd
- SW11 pad 2: Row1 -> gnd
- SW11_r1 pad 2: Row1 -> gnd
- SW12 pad 2: Row1 -> gnd
- SW12_r1 pad 2: Row2 -> gnd
- SW13_r1 pad 2: Row2 -> gnd
- SW14 pad 2: Row2 -> gnd
- SW14_r1 pad 2: Row2 -> gnd
- SW15 pad 2: Row2 -> gnd
- SW15_r1 pad 2: Row2 -> gnd
- SW16 pad 2: Row2 -> gnd
- SW16_r1 pad 2: Row2 -> gnd
- SW17 pad 2: Row2 -> gnd
- SW17_r1 pad 2: Row3 -> gnd
- SW18 pad 2: Row2 -> gnd
- SW18_r1 pad 2: Row3 -> gnd
- SW2 pad 2: Row0 -> gnd
- SW20 pad 2: Row3 -> gnd
- SW21 pad 2: Row3 -> gnd
- SW2_r1 pad 2: Row0 -> gnd
- SW3 pad 2: Row0 -> gnd
- SW3_r1 pad 2: Row0 -> gnd
- SW4 pad 2: Row0 -> gnd
- SW4_r1 pad 2: Row0 -> gnd
- SW5 pad 2: Row0 -> gnd
- SW5_r1 pad 2: Row0 -> gnd
- SW6 pad 2: Row0 -> gnd
- SW6_r1 pad 2: Row0 -> gnd
- SW7_r1 pad 2: Row1 -> gnd
- SW8 pad 2: Row1 -> gnd
- SW8_r1 pad 2: Row1 -> gnd
- SW9 pad 2: Row1 -> gnd
- SW9_r1 pad 2: Row1 -> gnd
- U1 pad 1: Column3 -> unconnected-(U1-Pad1)
- U1 pad 10: Column1 -> Switch17
- U1 pad 11: Column0 -> Switch18
- U1 pad 12: D+ -> Enc_A
- U1 pad 13: D- -> Enc_B
- U1 pad 14: gnd -> unconnected-(U1-Pad14)
- U1 pad 15: vcc -> unconnected-(U1-Pad15)
- U1 pad 2: Column4 -> unconnected-(U1-Pad2)
- U1 pad 3: Serial -> unconnected-(U1-Pad3)
- U1 pad 4: Row0 -> unconnected-(U1-Pad4)
- U1 pad 5: Row1 -> unconnected-(U1-Pad5)
- U1 pad 6: reset -> unconnected-(U1-Pad6)
- U1 pad 7: Row2 -> NRST
- U1 pad 8: Row3 -> gnd
- U1 pad 9: Column2 -> +3.3V
Routing:
- net Column0: track 165.9 -> 0.00 mm
- net Column1: track 152.9 -> 0.00 mm
- net Row0: track 134.0 -> 0.00 mm, vias 1 -> 0
- net Column2: track 133.9 -> 0.00 mm
- net Row1: track 123.6 -> 0.00 mm, vias 1 -> 0
- net Row2: track 121.8 -> 0.00 mm, vias 1 -> 0
- net +5V: track 0.00 -> 105.6 mm
- net Column3: track 99.8 -> 0.00 mm
- net Switch18: track 0.00 -> 88.2 mm, vias 0 -> 1
- net D+: track 4.53 -> 81.7 mm, vias 0 -> 2
- net Switch5: track 10.4 -> 87.1 mm
- net Row3: track 75.8 -> 0.00 mm, vias 1 -> 0
- net D-: track 4.53 -> 78.0 mm
- net Enc_A: track 0.00 -> 72.8 mm, vias 0 -> 1
- net Enc_B: track 0.00 -> 68.9 mm, vias 0 -> 1
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- added copper zone on B.Cu, net gnd
Other:
- board text removed: "Face down"
- board text removed: "Face up"
